File: IR-main/shift_register_PCB/communication_module_PCB_27_03_2024/communication_module_PCB.kicad_sch (KiCad schematic)
At the start: 47 parts

Commit message: PCB desing updated & Datasheets
Parts:
- removed D? (x4): LED, symbol Device:LED
- removed D? (x8): DIODE, symbol pspice:DIODE
- removed R?: 10k, symbol Device:R
- added C?: 47uF, symbol Device:C_Polarized
- added C?: 100nF, symbol pspice:CAP
- added D? (x13): LED, symbol Device:LED
- added Q? (x9): BC548, Package_TO_SOT_THT:TO-92_Inline, symbol Transistor_BJT:BC548
- added R? (x8): 33k, symbol Device:R
- added R?: 330, symbol Device:R
- added R?: 10k, symbol Device:R
- added R?: 2.2k, symbol Device:R
- added R?: 1k, symbol Device:R
- R?: value 10k -> 70
Connections:
- net 5V: now also C?.1, C?.1, R?.1, R?.1, R?.2
- net GND: now also C?.2, C?.2, Q?.3 (E), Q?.3 (E), Q?.3 (E), Q?.3 (E), Q?.3 (E), Q?.3 (E), Q?.3 (E), Q?.3 (E), Q?.3 (E)
- net IR_RECEIVER_OUTPUT: now also Q?.1 (C), Q?.1 (C), Q?.1 (C), Q?.1 (C), Q?.1 (C), Q?.1 (C), Q?.1 (C), Q?.1 (C), R?.1, R?.2
- net at D?.1 (K), Q?.1 (C): now also D?.1 (K) (x4)
- net at D?.2 (A), D?.2 (A), D?.2 (A)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: now also D?.2 (A), D?.2 (A), D?.2 (A), D?.2 (A)
- net at Q?.1 (C): now also D?.1 (K), D?.1 (K) (x4)
- net at U?.6: now also R?.2 (x2)
- net at U?.3: now also R?.2 (x2)
- net at U?.8: now also R?.2 (x2)
- net at U?.11: now also R?.2 (x2)
- new net: Q?.2 (B), R?.1 (x8)
- new net: D?.2 (A), D?.2 (A), D?.2 (A), D?.2 (A), D?.2 (A), D?.2 (A), D?.2 (A), R?.1
- new net: D?.2 (A), R?.2
- new net: D?.1 (K), Q?.1 (C)
- new net: Q?.2 (B), R?.2
Other:
- note added: "Results in 30mA current ( 5-0.7-0.7-1.5 = 2.1V drop) 30mA = 2.1V / 70 ohm"
- moved on the sheet: U?A, U?B, U?C, U?D, U?E

Commit message: Sensory-sensory approach first PCB
Parts:
- removed D? (x9): LED, symbol Device:LED
- removed Q? (x18): BC548, Package_TO_SOT_THT:TO-92_Inline, symbol Transistor_BJT:BC548
- removed R?: 330, symbol Device:R
- removed R?: 10k, symbol Device:R
- removed R?: 2.2k, symbol Device:R
- added QL0, QL1, QL2, QL3, QL4, QL5, QL6, QL7, QR0, QR1, QR2, QR3, QR4, QR5, QR6, QR7, QTr1: BC847, Package_TO_SOT_SMD:SOT-23, symbol Transistor_BJT:BC847
- added REC0, REC1, REC2, REC3, REC4, REC5, REC6, REC7: IR_REC, communication_library_pcb:IR-receiver, symbol communication_library_pcb:IR-receiver
- added U4: header-6, communication_library_pcb:header6, symbol communication_library_pcb:header-6
- C1: renamed from C?; footprint (none) -> Capacitor_SMD:C_Elec_6.3x5.4
- C2: renamed from C?; footprint (none) -> Capacitor_SMD:C_1206_3216Metric
- LED0, LED1, LED2, LED3, LED4, LED5, LED6, LED7: renamed from D?; footprint (none) -> LED_THT:LED_D3.0mm
- R-IR1, R12, R13, R14, R15, R18, R19, R20, R21, R22, RL0, RL1, RL2, RL3, RL4, RL5, RL6, RL7: renamed from R?; footprint (none) -> Resistor_SMD:R_1206_3216Metric_Pad1.30x1.75mm_HandSolder
- R5: renamed from R?; value 10k -> 1k; footprint (none) -> Resistor_SMD:R_1206_3216Metric_Pad1.30x1.75mm_HandSolder
- U1, U2, U3: renamed from U?; footprint (none) -> Package_DIP:DIP-14_W7.62mm
Connections:
- net 5V: now also REC0.3 (VCC), REC1.3 (VCC), REC2.3 (VCC), REC3.3 (VCC), REC4.3 (VCC), REC5.3 (VCC), REC6.3 (VCC), REC7.3 (VCC), U4.1 (5V)
- net CLOCK: now also U4.4 (CLK)
- net DATA: now also U4.3 (DATA)
- net GND: now also QR0.2 (E), QR1.2 (E), QR2.2 (E), QR3.2 (E), QR4.2 (E), QR5.2 (E), QR6.2 (E), QR7.2 (E), QTr1.2 (E), REC0.2 (GND), REC1.2 (GND), REC2.2 (GND), REC3.2 (GND), REC4.2 (GND), REC5.2 (GND), REC6.2 (GND), REC7.2 (GND), U4.2 (GND)
- net IR_RECEIVER_OUTPUT: now also QR0.3 (C), QR1.3 (C), QR2.3 (C), QR3.3 (C), QR4.3 (C), QR5.3 (C), QR6.3 (C), QR7.3 (C), U4.6 (R)
- net IR_REC_0: now also REC0.1 (OUT)
- net IR_REC_1: now also REC1.1 (OUT)
- net IR_REC_2: now also REC2.1 (OUT)
- net IR_REC_3: now also REC3.1 (OUT)
- net IR_REC_4: now also REC4.1 (OUT)
- net IR_REC_5: now also REC5.1 (OUT)
- net IR_REC_6: now also REC6.1 (OUT)
- net IR_REC_7: now also REC7.1 (OUT)
- net S0: now also U1.6 (Q3); no longer U1.3 (Q0)
- net S1: now also U1.5 (Q2); no longer U1.4 (Q1)
- net S2: now also U1.4 (Q1); no longer U1.5 (Q2)
- net S3: now also U1.3 (Q0); no longer U1.6 (Q3)
- net S4: now also U1.13 (Q7); no longer U1.10 (Q4)
- net S5: now also U1.12 (Q6); no longer U1.11 (Q5)
- net S6: now also U1.11 (Q5); no longer U1.12 (Q6)
- net S7: now also U1.10 (Q4); no longer U1.13 (Q7)
- net TRANSMIT: now also U4.5 (T)
- net at R19.1: now also QR4.1 (B)
- net at RL4.1: now also QL4.1 (B)
- net at LED6.1 (K): now also QL6.3 (C)
- net at LED2.1 (K): now also QL2.3 (C)
- net at RL2.1: now also QL2.1 (B)
- net at LED7.1 (K): now also QL7.3 (C)
- net at R14.1: now also QR2.1 (B)
- net at LED0.1 (K): now also QL0.3 (C)
- net at RL0.1: now also QL0.1 (B)
- net at R21.1: now also QR6.1 (B)
- net at R12.1: now also QR0.1 (B)
- net at LED4.1 (K): now also QL4.3 (C)
- net at LED3.1 (K): now also QL3.3 (C)
- net at R22.1: now also QR7.1 (B)
- net at R13.1: now also QR1.1 (B)
- net at LED1.1 (K): now also QL1.3 (C)
- net at R5.2: now also QTr1.1 (B)
- net at RL7.1: now also QL7.1 (B)
- net at RL1.1: now also QL1.1 (B)
- net at R20.1: now also QR5.1 (B)
- net at RL5.1: now also QL5.1 (B)
- net at R15.1: now also QR3.1 (B)
- net at RL3.1: now also QL3.1 (B)
- net at LED5.1 (K): now also QL5.3 (C)
- net at RL6.1: now also QL6.1 (B)
- new net: QL0.2 (E), QL1.2 (E), QL2.2 (E), QL3.2 (E), QL4.2 (E), QL5.2 (E), QL6.2 (E), QL7.2 (E), QTr1.3 (C)
Other:
- note added: "Results in 30mA current ( 5-0.2-0.2-1.5 = 3.1V drop) 30mA = 3.1V / 100 ohm"
- note removed: "Results in 30mA current ( 5-0.7-0.7-1.5 = 2.1V drop) 30mA = 2.1V / 70 ohm"
- moved on the sheet: R-IR1
